Commit message: new spot.urdf

File: horizon/examples/urdf/spot.urdf (robot description, URDF)
Before this commit: robot spot, 20 links, 19 joints
Links:
- link base_link: geometry collision mesh filename=package://spot_urdf/meshes/body_collision.stl; visual mesh filename=package://spot_urdf/meshes/body.dae
- link lf_hip: geometry collision mesh filename=package://spot_urdf/meshes/front_left_hip_collision.stl; visual mesh filename=package://spot_urdf/meshes/front_left_hip.dae
- link lf_lowerleg: geometry collision mesh filename=package://spot_urdf/meshes/front_left_lower_leg_collision.s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; visual mesh filename=package://spot_urdf/meshes/front_left_lower_leg.dae
- link lf_upperleg: geometry collision mesh filename=package://spot_urdf/meshes/front_left_upper_leg_collision.s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; visual mesh filename=package://spot_urdf/meshes/front_left_upper_leg.dae
- link lh_hip: geometry collision mesh filename=package://spot_urdf/meshes/rear_left_hip_collision.stl; visual mesh filename=package://spot_urdf/meshes/rear_left_hip.dae
- link lh_lowerleg: geometry collision mesh filename=package://spot_urdf/meshes/rear_left_lower_leg_collision.stl; visual mesh filename=package://spot_urdf/meshes/rear_left_lower_leg.dae
- link lh_upperleg: geometry collision mesh filename=package://spot_urdf/meshes/rear_left_upper_leg_collision.stl; visual mesh filename=package://spot_urdf/meshes/rear_left_upper_leg.dae
- link rf_hip: geometry collision mesh filename=package://spot_urdf/meshes/front_right_hip_collision.stl; visual mesh filename=package://spot_urdf/meshes/front_right_hip.dae
- link rf_lowerleg: geometry collision mesh filename=package://spot_urdf/meshes/front_right_lower_leg_collision.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; visual mesh filename=package://spot_urdf/meshes/front_right_lower_leg.dae
- link rf_upperleg: geometry collision mesh filename=package://spot_urdf/meshes/front_right_upper_leg_collision.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; visual mesh filename=package://spot_urdf/meshes/front_right_upper_leg.dae
- link rh_hip: geometry collision mesh filename=package://spot_urdf/meshes/rear_right_hip_collision.stl; visual mesh filename=package://spot_urdf/meshes/rear_right_hip.dae
- link rh_lowerleg: geometry collision mesh filename=package://spot_urdf/meshes/rear_right_lower_leg_collision.s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; visual mesh filename=package://spot_urdf/meshes/rear_right_lower_leg.dae
- link rh_upperleg: geometry collision mesh filename=package://spot_urdf/meshes/rear_right_upper_leg_collision.s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; visual mesh filename=package://spot_urdf/meshes/rear_right_upper_leg.dae
Joints:
- joint lf_foot_joint: origin xyz=-0.01 0.0 -0.35 rpy=0 0 0 -> xyz=-0.005 0.0 -0.348 rpy=0 0 0
- joint lh_foot_joint: origin xyz=-0.01 0.0 -0.35 rpy=0 0 0 -> xyz=-0.005 0.0 -0.348 rpy=0 0 0
- joint rf_foot_joint: origin xyz=-0.01 0.0 -0.35 rpy=0 0 0 -> xyz=-0.005 0.0 -0.348 rpy=0 0 0
- joint rh_foot_joint: origin xyz=-0.01 0.0 -0.35 rpy=0 0 0 -> xyz=-0.005 0.0 -0.348 rpy=0 0 0

Commit message: lapacke ldlt and others

File: horizon/examples/urdf/spot.urdf (robot description, URDF)
Before this commit: robot spot, 20 links, 19 joints
Links:
- link lf_foot: geometry visual sphere radius=0.01
- link lh_foot: geometry visual sphere radius=0.01
- link rf_foot: geometry visual sphere radius=0.01
- link rh_foot: geometry visual sphere radius=0.01
Joints:
- joint lf_foot_joint: origin xyz=-0.005 0.0 -0.348 rpy=0 0 0 -> xyz=-0.005 0.0 -0.368 rpy=0 0 0
- joint lh_foot_joint: origin xyz=-0.005 0.0 -0.348 rpy=0 0 0 -> xyz=-0.005 0.0 -0.368 rpy=0 0 0
- joint rf_foot_joint: origin xyz=-0.005 0.0 -0.348 rpy=0 0 0 -> xyz=-0.005 0.0 -0.368 rpy=0 0 0
- joint rh_foot_joint: origin xyz=-0.005 0.0 -0.348 rpy=0 0 0 -> xyz=-0.005 0.0 -0.368 rpy=0 0 0

Commit message: checked out old spot_jump.mat and spot.urdf

File: horizon/examples/urdf/spot.urdf (robot description, URDF)
Before this commit: robot spot, 20 links, 19 joints
Links:
- link lf_foot: geometry collision sphere radius=0.03; visual sphere radius=0.019999999999999997
- link lh_foot: geometry collision sphere radius=0.03; visual sphere radius=0.019999999999999997
- link rf_foot: geometry collision sphere radius=0.03; visual sphere radius=0.019999999999999997
- link rh_foot: geometry collision sphere radius=0.03; visual sphere radius=0.019999999999999997
Joints:
- joint lf_foot_joint: origin xyz=-0.005 0.0 -0.368 rpy=0 0 0 -> xyz=-0.005 0.0 -0.348 rpy=0 0 0
- joint lh_foot_joint: origin xyz=-0.005 0.0 -0.368 rpy=0 0 0 -> xyz=-0.005 0.0 -0.348 rpy=0 0 0
- joint rf_foot_joint: origin xyz=-0.005 0.0 -0.368 rpy=0 0 0 -> xyz=-0.005 0.0 -0.348 rpy=0 0 0
- joint rh_foot_joint: origin xyz=-0.005 0.0 -0.368 rpy=0 0 0 -> xyz=-0.005 0.0 -0.348 rpy=0 0 0
