Commit message: still examples refactor

File: horizon/examples/urdf/quadruped_template.urdf (robot description, URDF)
Before this commit: robot template, 15 links, 14 joints
Joints:
- joint Contact1_x: limit lower=-1 upper=1 effort=0 velocity=1 -> lower=0.1 upper=0.6 effort=0 velocity=1
- joint Contact1_y: limit lower=-1 upper=1 effort=0 velocity=1 -> lower=0.1 upper=0.5 effort=0 velocity=1
- joint Contact1_z: limit lower=-1 upper=1 effort=0 velocity=1 -> lower=-0.635 upper=-0.435 effort=0 velocity=1
- joint Contact2_x: limit lower=-1 upper=1 effort=0 velocity=1 -> lower=0.1 upper=0.6 effort=0 velocity=1
- joint Contact2_y: limit lower=-1 upper=1 effort=0 velocity=1 -> lower=-0.5 upper=-0.1 effort=0 velocity=1
- joint Contact2_z: limit lower=-1 upper=1 effort=0 velocity=1 -> lower=-0.635 upper=-0.435 effort=0 velocity=1
- joint Contact3_x: limit lower=-1 upper=1 effort=0 velocity=1 -> lower=-0.6 upper=-0.1 effort=0 velocity=1
- joint Contact3_y: limit lower=-1 upper=1 effort=0 velocity=1 -> lower=-0.5 upper=-0.1 effort=0 velocity=1
- joint Contact3_z: limit lower=-1 upper=1 effort=0 velocity=1 -> lower=-0.635 upper=-0.435 effort=0 velocity=1
- joint Contact4_x: limit lower=-1 upper=1 effort=0 velocity=1 -> lower=-0.6 upper=-0.1 effort=0 velocity=1
- joint Contact4_y: limit lower=-1 upper=1 effort=0 velocity=1 -> lower=0.1 upper=0.5 effort=0 velocity=1
- joint Contact4_z: limit lower=-1 upper=1 effort=0 velocity=1 -> lower=-0.635 upper=-0.435 effort=0 velocity=1

File: horizon/examples/urdf/roped_template.urdf (robot description, URDF)
Before this commit: robot roped_template, 15 links, 14 joints
Joints:
- joint rope_joint: limit lower=0 upper=3 effort=0 velocity=10 -> lower=0 upper=10 effort=0 velocity=10
